File: Kicad_Mesh3310/nfc.kicad_sch (KiCad schematic)
At the start: 9 parts

Commit message: Cleaning and placing
Cleaning and placing components
Parts:
- AE1: footprint mesh3310:NFC_2.8uH_COIL -> mesh3310_footprints:NFC_2.8uH_COIL
- RF2: footprint lcsc:IPEX-SMD_3P-L2.6-W2.6-LS3.0_RF1200001R -> mesh3310_footprints:IPEX-SMD_3P-L2.6-W2.6-LS3.0_RF1200001R
Changed lines of the file:
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@@
 			)
 		)
-		(property "Footprint" "mesh3310:NFC_2.8uH_COIL"
+		(property "Footprint" "mesh3310_footprints:NFC_2.8uH_COIL"
 			(at 106.68 113.03 0)
 			(effects
@@
 			)
 		)
-		(property "Footprint" "lcsc:IPEX-SMD_3P-L2.6-W2.6-LS3.0_RF1200001R"
+		(property "Footprint" "mesh3310_footprints:IPEX-SMD_3P-L2.6-W2.6-LS3.0_RF1200001R"
 			(at 157.48 95.25 0)
 			(effects
