File: Kicad_Mesh3310/interfaces.kicad_sch (KiCad schematic)
At the start: 66 parts, among them J10 Speaker pad, J2 Mic pad, J5 Vibrator pad, J6 Buzzer pad, J7 Display, Q1 BC847, Q4 BSS138, Q5 BSS138, Q6 IRLML6401, Q7 BSS138, U5 MAX98357A

Commit message: Schema afgemaakt, 6-laags layout, LCSC-onderdelen en productiebestanden
- schema opgeschoond en aangevuld (ERC 0)
- bord naar 6 lagen (JLC06161H-3313), volledig gerouteerd, DRC 0
- LTE via U.FL, USB via bodemconnector J4
- LCSC-nummers voor alle onderdelen, datasheets toegevoegd
- gerbers, boorbestanden, positiebestand en stuklijst in productie/
Parts:
- C14, C18, C21: LCSC (none) -> C408130
- C15: LCSC (none) -> C384825
- C16: footprint Capacitor_Tantalum_SMD:CP_EIA-1608-08_AVX-J -> Capacitor_SMD:C_0603_1608Metric; symbol Device:C_Polarized -> Device:C; LCSC (none) -> C19702
- C17: value 47uF/10V -> 22uF/6.3V; footprint Capacitor_Tantalum_SMD:CP_EIA-1608-08_AVX-J -> Capacitor_SMD:C_0603_1608Metric; symbol Device:C_Polarized -> Device:C; LCSC (none) -> C59461
- C20: value 100uF -> 10uF/10V; footprint Capacitor_SMD:C_0201_0603Metric -> Capacitor_SMD:C_0603_1608Metric; LCSC (none) -> C19702
- D10, D11, D12, D13, D5, D6, D7, D9: LCSC (none) -> C2827254
- D4, D8: LCSC (none) -> C5355496
- Q1: LCSC (none) -> C57668
- Q4, Q5, Q7: LCSC (none) -> C518792
- Q6: LCSC (none) -> C22363750
- R15, R17, R20, R37: LCSC (none) -> C3152012
- R16: LCSC (none) -> C49654370
- R18, R31, R32, R33, R34, R35: LCSC (none) -> C304544
- R19, R21, R22, R23, R24, R25, R26, R27: value 56R -> 150R; LCSC (none) -> C49653085
- R30: LCSC (none) -> C3152038
- R36: LCSC (none) -> C49653410
- R38: LCSC (none) -> C473473
- R9: LCSC (none) -> C171950
- U5: LCSC (none) -> C910544
Connections:
- net P0.18_COL_3 renamed P0.19_COL_3
