File: Kicad_Mesh3310/interfaces.kicad_sch (KiCad schematic)
At the start: 66 parts, among them J10 Speaker pad, J2 Mic pad, J5 Vibrator pad, J6 Buzzer pad, J7 Display, Q1 BC847, Q4 BSS138, Q5 BSS138, Q6 IRLML6401, Q7 BSS138, U5 MAX98357A

Commit message: Rev. F + G: controleronde, TPS3420 aan/uit-knop, FLASH_CS pull-up, RF4 DNP, U.FL-variant LoRa
Parts:
- added R65: 100k, Resistor_SMD:R_0201_0603Metric, symbol Device:R
- D4, D8: value BAT60A -> 1N4148WS; LCSC C5355496 -> C2128
- Q4, Q7: value BSS138 -> AO3400A; LCSC C518792 -> C20917
- R36: value 220k -> 1M; LCSC C49653410 -> C473482
Connections:
- net GND: now also R65.1
- net ~{DISP_RST}: now also R65.2
Changed lines of the file:
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@@
 		(title "Mainboard replacement for Nokia 3310")
 		(date "29-12-2025")
-		(rev "Rev A")
+		(rev "Rev G")
 		(company "Mesh3310")
 		(comment 1 "JDJ electronics")
@@
 		)
 	)
+	(label "~{DISP_RST}"
+		(at 111.76 52.07 0)
+		(effects
+			(font
+				(size 1.27 1.27)
+			)
+			(justify left bottom)
+		)
+	)
 	(hierarchical_label "I2S_LRCK"
 		(shape bidirectional)
@@
 			)
 		)
-		(property "Value" "BSS138"
+		(property "Value" "AO3400A"
 			(at 256.54 58.42 0)
 			(effects
@@
 			)
 		)
-		(property "LCSC" "C518792"
+		(property "LCSC" "C20917"
 			(at 256.54 56.515 0)
 			(effects
@@
 			)
 		)
-		(property "Value" "220k"
+		(property "Value" "1M"
 			(at 245.11 134.6199 0)
 			(effects
@@
 			)
 		)
-		(property "LCSC" "C49653410"
+		(property "LCSC" "C473482"
 			(at 244.348 133.35 90)
 			(effects
@@
 	)
 	(symbol
+		(lib_id "Device:R")
+		(at 111.76 55.88 180)
+		(unit 1)
+		(exclude_from_sim no)
+		(in_bom yes)
+		(on_board yes)
+		(dnp no)
+		(fields_autoplaced yes)
+		(property "Reference" "R65"
+			(at 114.26 54.61 0)
+			(effects
+				(font
+					(size 1.27 1.27)
+				)
+				(justify right)
+			)
+		)
+		(property "Value" "100k"
+			(at 114.26 57.15 0)
+			(effects
+				(font
+					(size 1.27 1.27)
+				)
+				(justify right)
+			)
+		)
+		(property "Footprint" "Resistor_SMD:R_0201_0603Metric"
+			(at 113.54 55.88 90)
+			(effects
+				(font
+					(size 1.27 1.27)
+				)
+				(hide yes)
+			)
+		)
+		(property "LCSC" "C3152012"
+			(at 113.54 55.88 90)
+			(effects
+				(font
+					(size 1.27 1.27)
+				)
+				(hide yes)
+			)
+		)
+		(property "Datasheet" "~"
+			(at 111.76 55.88 0)
+			(effects
+				(font
+					(size 1.27 1.27)
+				)
+				(hide yes)
+			)
+		)
+		(property "Description" "Resistor"
+			(at 111.76 55.88 0)
+			(effects
+				(font
+					(size 1.27 1.27)
+				)
+				(hide yes)
+			)
+		)
+		(property "PN" "603-RC0402JR-13100KL"
+			(at 111.76 55.88 0)
+			(effects
+				(font
+					(size 1.27 1.27)
+				)
+				(hide yes)
+			)
+		)
+		(property "MPN" "603-RC0402JR-13100KL"
+			(at 111.76 55.88 0)
+			(effects
+				(font
+					(size 1.27 1.27)
+				)
+				(hide yes)
+			)
+		)
+		(pin "2"
+		)
+		(pin "1"
+		)
+		(instances
+			(project "Mesh3310"
+				(path "/8d65c5ef-7a02-4454-aee5-ab9c49e4aeab/56951be9-e7d0-42f1-a860-fb701fde1659"
+					(reference "R65")
+					(unit 1)
+				)
+			)
+		)
+	)
+	(symbol
+		(lib_id "power:GND")
+		(at 111.76 59.69 0)
+		(unit 1)
+		(exclude_from_sim no)
+		(in_bom yes)
+		(on_board yes)
+		(dnp no)
+		(fields_autoplaced yes)
+		(property "Reference" "#PWR0141"
+			(at 111.76 66.04 0)
+			(effects
+				(font
+					(size 1.27 1.27)
+				)
+				(hide yes)
+			)
+		)
+		(property "Value" "GND"
+			(at 111.76 64.77 0)
+			(effects
+				(font
+					(size 1.27 1.27)
+				)
+			)
+		)
+		(property "Footprint" ""
+			(at 111.76 59.69 0)
+			(effects
+				(font
+					(size 1.27 1.27)
+				)
+				(hide yes)
+			)
+		)
+		(property "Datasheet" ""
+			(at 111.76 59.69 0)
+			(effects
+				(font
+					(size 1.27 1.27)
+				)
+				(hide yes)
+			)
+		)
+		(property "Description" "Power symbol creates a global label with name \"GND\" , ground"
+			(at 111.76 59.69 0)
+			(effects
+				(font
+					(size 1.27 1.27)
+				)
+				(hide yes)
+			)
+		)
+		(pin "1"
+		)
+		(instances
+			(project "Mesh3310"
+				(path "/8d65c5ef-7a02-4454-aee5-ab9c49e4aeab/56951be9-e7d0-42f1-a860-fb701fde1659"
+					(reference "#PWR0141")
+					(unit 1)
+				)
+			)
+		)
+	)
+	(symbol
 		(lib_id "power:+3V3")
 		(at 156.21 43.18 0)
@@
 			)
 		)
-		(property "Value" "BAT60A"
+		(property "Value" "1N4148WS"
 			(at 263.652 44.0746 90)
 			(effects
@@
 			)
 		)
-		(property "LCSC" "C5355496"
+		(property "LCSC" "C2128"
 			(at 257.175 43.18 0)
 			(effects
@@
 			)
 		)
-		(property "Value" "BAT60A"
+		(property "Value" "1N4148WS"
 			(at 229.362 44.0746 90)
 			(effects
@@
 			)
 		)
-		(property "LCSC" "C5355496"
+		(property "LCSC" "C2128"
 			(at 222.885 43.18 0)
 			(effects
@@
 			)
 		)
-		(property "Value" "BSS138"
+		(property "Value" "AO3400A"
 			(at 222.25 58.42 0)
 			(effects
@@
 			)
 		)
-		(property "LCSC" "C518792"
+		(property "LCSC" "C20917"
 			(at 222.25 56.515 0)
 			(effects

Commit message: Onderdelen die JLC niet had vervangen, JLC-uploadbestanden toegevoegd
Parts:
- R9: LCSC C171950 -> C138109
Changed lines of the file:
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@@
 			)
 		)
-		(property "LCSC" "C171950"
+		(property "LCSC" "C138109"
 			(at 227.838 133.35 90)
 			(effects
