File: Kicad_Mesh3310/gnss.kicad_sch (KiCad schematic)
At the start: 26 parts, among them J3 Sim/Pad, J8 Conn_Coaxial, U12 nRF9151-LAXX, U2 MX25R1635FZNIH0, U6 SIM-ST-MFF2, U8 SKY65723-81

Commit message: Schema afgemaakt, 6-laags layout, LCSC-onderdelen en productiebestanden
- schema opgeschoond en aangevuld (ERC 0)
- bord naar 6 lagen (JLC06161H-3313), volledig gerouteerd, DRC 0
- LTE via U.FL, USB via bodemconnector J4
- LCSC-nummers voor alle onderdelen, datasheets toegevoegd
- gerbers, boorbestanden, positiebestand en stuklijst in productie/
Parts:
- added C93, C94: NC (afstemmen), Capacitor_SMD:C_0201_0603Metric, symbol Device:C
- added J11: GNSS antenne (U.FL), Connector_Coaxial:U.FL_Hirose_U.FL-R-SMT-1_Vertical, symbol Connector:Conn_Coaxial
- added R61: 0R, Resistor_SMD:R_0201_0603Metric, symbol Device:R_Small
- C10, C12, C2, C4: footprint Resistor_SMD:R_0201_0603Metric -> Capacitor_SMD:C_0201_0603Metric; LCSC (none) -> C408130
- C11: footprint Resistor_SMD:R_0201_0603Metric -> Capacitor_SMD:C_0201_0603Metric; LCSC (none) -> C5142550
- C13: LCSC C1525 -> C408130
- C26: LCSC (none) -> C5142550
- C28: value 47u -> 47uF/6.3V; footprint Capacitor_SMD:C_0201_0603Metric -> Capacitor_SMD:C_0805_2012Metric; LCSC (none) -> C16780
- C3: footprint Resistor_SMD:R_0201_0603Metric -> Capacitor_SMD:C_0402_1005Metric; LCSC (none) -> C23733
- C33, C43: LCSC (none) -> C408130
- C8: footprint Capacitor_SMD:C_0201_0603Metric -> Capacitor_SMD:C_0402_1005Metric; LCSC (none) -> C23733
- D1: LCSC (none) -> C19829475
- FB1: value 120 -> 120R@100MHz 1A; footprint Resistor_SMD:R_0201_0603Metric -> Inductor_SMD:L_0603_1608Metric; LCSC (none) -> C14709
- J8: value Conn_Coaxial -> LTE antenne: U.FL -> flexantenne (bv. Taoglas FXUB63); LCSC (none) -> C88374
- R10, R28: now not fitted
- R12: LCSC (none) -> C3152038
- R13, R29: LCSC (none) -> C3152043
- R14: LCSC (none) -> C473450
- U12: LCSC (none) -> C42236596
- U2: value MX25R1635FZNIH0 -> MX25R1635FZUIH0; footprint mesh3310_footprints:SON127P500X600X80-9N -> Package_SON:Winbond_USON-8-1EP_3x2mm_P0.5mm_EP0.2x1.6mm; LCSC (none) -> C5687033
- U8: LCSC (none) -> C2654196
Connections:
- net FLASH_RESET is gone; now on net +3V3: U2.7 (~{RESET}/SIO3)
- net FLASH_WP is gone; now on net +3V3: U2.3 (~{WP}/SIO2)
- net GND: now also U2.9 (EXP), C93.2, C94.2, J11.2 (Ext); no longer U12.26 (SIM_DET)
- net RF_ANT: now also C93.1, R61.1; no longer J8.1 (In)
- net SIM_CLK: no longer D1.5 (K)
- net SIM_IO: now also D1.5 (K)
- net RF_AUX: no longer names the net of U12.37 (AUX)
- net RF_AUX: no longer C11.2
- new net: C94.1, J8.1 (In), R61.2
- new net: C11.2, J11.1 (In)
- no-connect marks 0 -> 33
Other:
- note added: "LTE: flexantenne in de behuizing via U.FL J8 (LoRa houdt de antennezone bovenin). Pi-netwerk R61/C93/C94 afstemmen met de gekozen antenne + kabel."

Commit message: Rev. C: schemafixes uit datasheetcontrole (VDD-buffer nRF9151, DC-blok LoRa, DNP C70/C71/BT2, deler 1M, laadtimers aan)
Parts:
- added C95: 10u, Capacitor_SMD:C_0402_1005Metric, symbol Device:C
Connections:
- net GND: now also C95.2
- net at FB1.2, R12.1, U12.14 (VDD): now also C95.1
Changed lines of the file:
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@@
+	)
+	(junction
+		(at 177.8 58.42)
+		(diameter 0)
+		(color 0 0 0 0)
 	)
 	(junction
@@
 		(diameter 0)
 		(color 0 0 0 0)
+	)
+	(wire
+		(pts
+			(xy 177.8 58.42) (xy 177.8 59.69)
+		)
+		(stroke
+			(width 0)
+			(type default)
+		)
 	)
 	(wire
@@
 					(unit 1)
 				)
+			)
+		)
+	)
+	(symbol
+		(lib_id "Device:C")
+		(at 177.8 63.5 0)
+		(unit 1)
+		(exclude_from_sim no)
+		(in_bom yes)
+		(on_board yes)
+		(dnp no)
+		(property "Reference" "C95"
+			(at 180.975 62.23 0)
+			(effects
+				(font
+					(size 1.27 1.27)
+				)
+				(justify left)
+			)
+		)
+		(property "Value" "10u"
+			(at 180.975 64.77 0)
+			(effects
+				(font
+					(size 1.27 1.27)
+				)
+				(justify left)
+			)
+		)
+		(property "Footprint" "Capacitor_SMD:C_0402_1005Metric"
+			(at 178.7652 67.31 0)
+			(effects
+				(font
+					(size 1.27 1.27)
+				)
+				(hide yes)
+			)
+		)
+		(property "LCSC" "C15525"
+			(at 178.7652 67.31 0)
+			(effects
+				(font
+					(size 1.27 1.27)
+				)
+				(hide yes)
+			)
+		)
+		(property "Datasheet" ""
+			(at 177.8 63.5 0)
+			(effects
+				(font
+					(size 1.27 1.27)
+				)
+				(hide yes)
+			)
+		)
+		(property "Description" ""
+			(at 177.8 63.5 0)
+			(effects
+				(font
+					(size 1.27 1.27)
+				)
+				(hide yes)
+			)
+		)
+		(property "Voltage" ""
+			(at 180.975 67.31 0)
+			(effects
+				(font
+					(size 1.27 1.27)
+				)
+				(justify left)
+			)
+		)
+		(property "Manufacturer Part Number" ""
+			(at 177.8 63.5 0)
+			(effects
+				(font
+					(size 1.27 1.27)
+				)
+				(hide yes)
+			)
+		)
+		(property "Part Number" ""
+			(at 177.8 63.5 0)
+			(effects
+				(font
+					(size 1.27 1.27)
+				)
+				(hide yes)
+			)
+		)
+		(property "Circuit Dojo PN" ""
+			(at 177.8 63.5 0)
+			(effects
+				(font
+					(size 1.27 1.27)
+				)
+				(hide yes)
+			)
+		)
+		(pin "1"
+		)
+		(pin "2"
+		)
+		(instances
+			(project "Mesh3310"
+				(path "/8d65c5ef-7a02-4454-aee5-ab9c49e4aeab/98e1aac4-af48-4762-9c2a-9b5d76c64f4f"
+					(reference "C95")
+					(unit 1)
+				)
+			)
+		)
+	)
+	(symbol
+		(lib_id "power:GND")
+		(at 177.8 67.31 0)
+		(unit 1)
+		(exclude_from_sim no)
+		(in_bom yes)
+		(on_board yes)
+		(dnp no)
+		(fields_autoplaced yes)
+		(property "Reference" "#PWR0133"
+			(at 177.8 73.66 0)
+			(effects
+				(font
+					(size 1.27 1.27)
+				)
+				(hide yes)
+			)
+		)
+		(property "Value" "GND"
+			(at 177.8 72.39 0)
+			(effects
+				(font
+					(size 1.27 1.27)
+				)
+			)
+		)
+		(property "Footprint" ""
+			(at 177.8 67.31 0)
+			(effects
+				(font
+					(size 1.27 1.27)
+				)
+				(hide yes)
+			)
+		)
+		(property "Datasheet" ""
+			(at 177.8 67.31 0)
+			(effects
+				(font
+					(size 1.27 1.27)
+				)
+				(hide yes)
+			)
+		)
+		(property "Description" "Power symbol creates a global label with name \"GND\" , ground"
+			(at 177.8 67.31 0)
+			(effects
+				(font
+					(size 1.27 1.27)
+				)
+				(hide yes)
+			)
+		)
+		(pin "1"
+		)
+		(instances
+			(project "Mesh3310"
+				(path "/8d65c5ef-7a02-4454-aee5-ab9c49e4aeab/98e1aac4-af48-4762-9c2a-9b5d76c64f4f"
+					(reference "#PWR0133")
+					(unit 1)
+				)

Commit message: Rev. D/E: nRF9151 op VSYS, aan/uit-knop kort=firmware lang=uit, 3V3 na ENABLE, buffer VSYS
Connections:
- net +3V3: no longer FB1.1
- net at C95.1, FB1.2, U12.14 (VDD): no longer R12.1
- new net PWR_EN: R12.1
- new net VSYS: FB1.1
Changed lines of the file:
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@@
+		)
+	)
+	(global_label "VSYS"
+		(shape passive)
+		(at 154.94 58.42 180)
+		(fields_autoplaced yes)
+		(effects
+			(font
+				(size 1.27 1.27)
+			)
+			(justify right)
+		)
+		(property "Intersheetrefs" "${INTERSHEET_REFS}"
+			(at 154.94 58.42 0)
+			(effects
+				(font
+					(size 1.27 1.27)
+				)
+				(justify right)
+				(hide yes)
+			)
+		)
+	)
+	(global_label "PWR_EN"
+		(shape passive)
+		(at 154.94 69.85 90)
+		(fields_autoplaced yes)
+		(effects
+			(font
+				(size 1.27 1.27)
+			)
+			(justify left)
+		)
+		(property "Intersheetrefs" "${INTERSHEET_REFS}"
+			(at 154.94 69.85 0)
+			(effects
+				(font
+					(size 1.27 1.27)
+				)
+				(justify left)
+				(hide yes)
+			)
 		)
 	)
@@
 	)
 	(junction
-		(at 168.91 58.42)
-		(diameter 0)
-		(color 0 0 0 0)
-	)
-	(junction
 		(at 151.13 58.42)
 		(diameter 0)
@@
 	(wire
 		(pts
+			(xy 154.94 58.42) (xy 157.48 58.42)
+		)
+		(stroke
+			(width 0)
+			(type default)
+		)
+	)
+	(wire
+		(pts
 			(xy 177.8 58.42) (xy 177.8 59.69)
 		)
@@
 	(wire
 		(pts
-			(xy 151.13 58.42) (xy 157.48 58.42)
-		)
-		(stroke
-			(width 0)
-			(type default)
-		)
-	)
-	(wire
-		(pts
 			(xy 143.51 187.96) (xy 157.48 187.96)
 		)
@@
 		(pts
 			(xy 152.4 127) (xy 157.48 127)
-		)
-		(stroke
-			(width 0)
-			(type default)
-		)
-	)
-	(wire
-		(pts
-			(xy 154.94 69.85) (xy 168.91 69.85)
 		)
 		(stroke
@@
 		)
 		(stroke
-			(width 0)
-			(type default)
-		)
-	)
-	(wire
-		(pts
-			(xy 168.91 69.85) (xy 168.91 58.42)
-		)
-		(stroke

Commit message: Rev. F + G: controleronde, TPS3420 aan/uit-knop, FLASH_CS pull-up, RF4 DNP, U.FL-variant LoRa
Parts:
- added R66: 100k, Resistor_SMD:R_0201_0603Metric, symbol Device:R
- C12: now not fitted; now left out of the parts list
- R14: value 1M -> 100k; LCSC C473450 -> C3152012
Connections:
- net +3V3: now also R66.1; no longer C2.1, C26.1, C28.1
- net FLASH_CS: now also R66.2
- net VDD_9151: now reaches C95.1, FB1.2, U12.14 (VDD)
- net VDD_9151: now also C2.1, C26.1, C28.1
Changed lines of the file:
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@@
 		(title "Mainboard replacement for Nokia 3310")
 		(date "29-12-2025")
-		(rev "Rev A")
+		(rev "Rev G")
 		(company "Mesh3310")
 		(comment 1 "JDJ electronics")
@@
 	(wire
 		(pts
-			(xy 130.81 55.88) (xy 130.81 58.42)
-		)
-		(stroke
-			(width 0)
-			(type default)
-		)
-	)
-	(wire
-		(pts
 			(xy 337.82 132.08) (xy 337.82 106.68)
 		)
@@
 		)
 	)
+	(label "FLASH_CS"
+		(at 124.46 237.49 0)
+		(effects
+			(font
+				(size 1.27 1.27)
+			)
+			(justify left bottom)
+		)
+	)
+	(label "VDD_9151"
+		(at 151.13 58.42 0)
+		(effects
+			(font
+				(size 1.27 1.27)
+			)
+			(justify left bottom)
+		)
+	)
+	(label "VDD_9151"
+		(at 182.88 58.42 0)
+		(effects
+			(font
+				(size 1.27 1.27)
+			)
+			(justify left bottom)
+		)
+	)
 	(label "SIM_VCC"
 		(at 101.6 190.5 0)
@@
 			)
 		)
-		(property "Value" "1M"
+		(property "Value" "100k"
 			(at 261.62 146.05 0)
 			(effects
@@
 			)
 		)
-		(property "LCSC" "C473450"
+		(property "LCSC" "C3152012"
 			(at 265.938 144.78 90)
 			(effects
@@
 	)
 	(symbol
+		(lib_id "Device:R")
+		(at 124.46 233.68 0)
+		(mirror y)
+		(unit 1)
+		(exclude_from_sim no)
+		(in_bom yes)
+		(on_board yes)
+		(dnp no)
+		(property "Reference" "R66"
+			(at 121.92 232.41 0)
+			(effects
+				(font
+					(size 1.27 1.27)
+				)
+				(justify left)
+			)
+		)
+		(property "Value" "100k"
+			(at 121.92 234.95 0)
+			(effects
+				(font
+					(size 1.27 1.27)
+				)
+				(justify left)
+			)
+		)
+		(property "Footprint" "Resistor_SMD:R_0201_0603Metric"
+			(at 126.24 233.68 90)
+			(effects
+				(font
+					(size 1.27 1.27)
+				)
+				(hide yes)
+			)
+		)
+		(property "LCSC" "C3152012"
+			(at 126.24 233.68 90)
+			(effects
+				(font
+					(size 1.27 1.27)
+				)
+				(hide yes)
+			)
+		)
+		(property "Datasheet" "~"
+			(at 124.46 233.68 0)
+			(effects
+				(font
+					(size 1.27 1.27)
+				)
+				(hide yes)
+			)
+		)
+		(property "Description" "Resistor"
+			(at 124.46 233.68 0)
+			(effects
+				(font
+					(size 1.27 1.27)
+				)
+				(hide yes)
+			)
+		)
+		(property "Tolerance" "1%"
+			(at 121.92 237.49 0)
+			(effects
+				(font
+					(size 1.27 1.27)
+				)
+				(justify left)
+			)
+		)
+		(property "Manufacturer Part Number" ""
+			(at 124.46 233.68 0)
+			(effects
+				(font
+					(size 1.27 1.27)
+				)
+				(hide yes)
+			)
+		)
+		(property "Part Number" "RES-100K-1%-02-0402"
+			(at 124.46 233.68 0)
+			(effects
+				(font
+					(size 1.27 1.27)
+				)
+				(hide yes)
+			)
+		)
+		(property "Circuit Dojo PN" "RES-1M-5%-0402"
+			(at 124.46 233.68 0)
+			(effects
+				(font
+					(size 1.27 1.27)
+				)
+				(hide yes)
+			)
+		)
+		(pin "1"
+		)
+		(pin "2"
+		)
+		(instances
+			(project "Mesh3310"
+				(path "/8d65c5ef-7a02-4454-aee5-ab9c49e4aeab/98e1aac4-af48-4762-9c2a-9b5d76c64f4f"
+					(reference "R66")
+					(unit 1)
+				)
+			)
+		)
+	)
+	(symbol
+		(lib_id "power:+3V3")
+		(at 124.46 229.87 0)
+		(unit 1)
+		(exclude_from_sim no)
+		(in_bom yes)
+		(on_board yes)
+		(dnp no)
+		(fields_autoplaced yes)
+		(property "Reference" "#PWR0148"
+			(at 124.46 233.68 0)
+			(effects
+				(font
+					(size 1.27 1.27)
+				)
+				(hide yes)
+			)
+		)
+		(property "Value" "+3V3"
+			(at 124.46 224.79 0)
+			(effects
+				(font
+					(size 1.27 1.27)
+				)
+			)
+		)
+		(property "Footprint" ""
+			(at 124.46 229.87 0)
+			(effects
+				(font
+					(size 1.27 1.27)
+				)
+				(hide yes)
+			)
+		)
+		(property "Datasheet" ""
+			(at 124.46 229.87 0)
+			(effects
+				(font
+					(size 1.27 1.27)
+				)
+				(hide yes)
+			)
+		)
+		(property "Description" "Power symbol creates a global label with name \"+3V3\""
+			(at 124.46 229.87 0)
+			(effects
+				(font
+					(size 1.27 1.27)
+				)
+				(hide yes)
+			)
+		)
+		(pin "1"
+		)
+		(instances
+			(project "Mesh3310"
+				(path "/8d65c5ef-7a02-4454-aee5-ab9c49e4aeab/98e1aac4-af48-4762-9c2a-9b5d76c64f4f"
+					(reference "#PWR0148")
+					(unit 1)
+				)
+			)
+		)
+	)
+	(symbol
 		(lib_id "Power_Protection:SP0504BAHT")
 		(at 88.9 209.55 0)
@@
 	)
 	(symbol
-		(lib_id "nrf91-feather-eagle-import:+3V3")
-		(at 130.81 53.34 0)
-		(mirror y)
-		(unit 1)
-		(exclude_from_sim no)
-		(in_bom yes)
-		(on_board yes)
-		(dnp no)
-		(property "Reference" "#+3V01"
-			(at 130.81 53.34 0)
-			(effects
-				(font
-					(size 1.27 1.27)
-				)
-				(hide yes)
-			)
-		)
-		(property "Value" "+3V3"
-			(at 133.35 50.8 0)
-			(effects
-				(font
-					(size 1.778 1.5113)
-				)
-				(justify left bottom)
-			)
-		)
-		(property "Footprint" ""
-			(at 130.81 53.34 0)
-			(effects
-				(font
-					(size 1.27 1.27)
-				)
-				(hide yes)
-			)
-		)
-		(property "Datasheet" ""
-			(at 130.81 53.34 0)
-			(effects
-				(font
-					(size 1.27 1.27)
-				)
-				(hide yes)
-			)
-		)
-		(property "Description" ""
-			(at 130.81 53.34 0)
-			(effects
-				(font
-					(size 1.27 1.27)
-				)
-				(hide yes)
-			)
-		)
-		(pin "1"
-		)
-		(instances
-			(project "Mesh3310"
-				(path "/8d65c5ef-7a02-4454-aee5-ab9c49e4aeab/98e1aac4-af48-4762-9c2a-9b5d76c64f4f"
-					(reference "#+3V01")
-					(unit 1)
-				)
-			)
-		)
-	)
-	(symbol
 		(lib_id "nrf91-feather-eagle-import:GND")
 		(at 190.5 219.71 0)
@@
 		(unit 1)
 		(exclude_from_sim no)
-		(in_bom yes)
+		(in_bom no)
 		(on_board yes)
-		(dnp no)
+		(dnp yes)
 		(property "Reference" "C12"
 			(at 271.145 143.51 0)
