File: Kicad_Mesh3310/rf.kicad_sch (KiCad schematic)
At the start: 34 parts, among them U1 TPE4259-63, U10 SX1262IMLTRT, X1 S201632M10PF10PPM 32MHz

Commit message: Schema afgemaakt, 6-laags layout, LCSC-onderdelen en productiebestanden
- schema opgeschoond en aangevuld (ERC 0)
- bord naar 6 lagen (JLC06161H-3313), volledig gerouteerd, DRC 0
- LTE via U.FL, USB via bodemconnector J4
- LCSC-nummers voor alle onderdelen, datasheets toegevoegd
- gerbers, boorbestanden, positiebestand en stuklijst in productie/
Parts:
- ANT1: LCSC (none) -> C3284550
- C19: LCSC C1623 -> C7393835
- C69: LCSC C1525 -> C408130
- C70, C71: LCSC C32949 -> C387913
- C75, C84: LCSC C22374861 -> C22374841
- C76: LCSC C82219 -> C301920
- C77: LCSC C472454 -> C881877
- C78: LCSC C48346 -> C1853504
- C79, C80: value C_Small -> NC
- C81: LCSC C41361091 -> C501815
- C82: LCSC C16193755 -> C526923
- C83: LCSC C86288 -> C285092
- C85, C86: LCSC C1523 -> C66942
- C87, C88: LCSC C161321 -> C301911
- C9: LCSC C5199872 -> C15849
- L13: LCSC C381880 -> C52109780
- L15: LCSC C17168 -> C473473
- L16: LCSC C27151 -> C46607399
- L17: LCSC C778764 -> C52109745
- L18: LCSC C86065 -> C52109761
- L19: LCSC C98003 -> C52109772
- L3: footprint Inductor_SMD:L_0201_0603Metric -> Inductor_SMD:L_0603_1608Metric
- R44, R45: LCSC C25076 -> C3152013
- R6: LCSC C25076 -> C473473
Changed lines of the file:
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@@
 			)
 		)
-		(property "LCSC" "C161321"
+		(property "LCSC" "C301911"
 			(at 259.08 95.25 0)
 			(effects
@@
 			)
 		)
-		(property "LCSC" "C86288"
+		(property "LCSC" "C285092"
 			(at 179.07 82.55 90)
 			(effects
@@
 			)
 		)
-		(property "LCSC" "C16193755"
+		(property "LCSC" "C526923"
 			(at 172.72 88.9 0)
 			(effects
@@
 			)
 		)
-		(property "LCSC" "C41361091"
+		(property "LCSC" "C501815"
 			(at 166.37 72.39 90)
 			(effects
@@
 			)
 		)
-		(property "LCSC" "C82219"
+		(property "LCSC" "C301920"
 			(at 139.7 72.39 90)
 			(effects
@@
 			)
 		)
-		(property "Footprint" "Inductor_SMD:L_0201_0603Metric"
+		(property "Footprint" "Inductor_SMD:L_0603_1608Metric"
 			(at 48.26 102.87 0)
 			(effects
@@
 			)
 		)
-		(property "LCSC" "C22374861"
+		(property "LCSC" "C22374841"
 			(at 138.43 113.03 0)
 			(effects
@@
 			)
 		)
-		(property "LCSC" "C472454"
+		(property "LCSC" "C881877"
 			(at 146.05 72.39 90)
 			(effects
@@
 			)
 		)
-		(property "LCSC" "C17168"
+		(property "LCSC" "C473473"
 			(at 143.51 82.55 90)
 			(effects
@@
 			)
 		)
-		(property "LCSC" "C25076"
+		(property "LCSC" "C3152013"
 			(at 215.9 109.22 90)
 			(effects
@@
 			)
 		)
-		(property "LCSC" "C25076"
+		(property "LCSC" "C473473"
 			(at 232.41 90.17 90)
 			(effects
@@
 			)
 		)
-		(property "LCSC" "C5199872"
+		(property "LCSC" "C15849"
 			(at 31.75 110.49 0)
 			(effects
@@
 			)
 		)
-		(property "LCSC" "C1523"
+		(property "LCSC" "C66942"
 			(at 220.98 114.3 0)
 			(effects
@@
 			)
 		)
-		(property "LCSC" "C98003"
+		(property "LCSC" "C52109772"
 			(at 255.27 90.17 90)
 			(effects
@@
 			)
 		)
-		(property "LCSC" "C32949"
+		(property "LCSC" "C387913"
 			(at 76.2 135.89 0)
 			(effects
@@
 			)
 		)
-		(property "LCSC" "C1525"
+		(property "LCSC" "C408130"
 			(at 62.23 111.76 90)
 			(effects
@@
 			)
 		)
-		(property "LCSC" "C27151"
+		(property "LCSC" "C46607399"
 			(at 151.13 73.66 0)
 			(effects
@@
 			)
 		)
-		(property "LCSC" "C25076"
+		(property "LCSC" "C3152013"
 			(at 215.9 64.77 90)
 			(effects
@@
 			)
 		)
-		(property "LCSC" "C48346"
+		(property "LCSC" "C1853504"
 			(at 151.13 102.87 90)
 			(effects
@@
 			)
 		)
-		(property "LCSC" "C1523"
+		(property "LCSC" "C66942"
 			(at 220.98 69.85 0)
 			(effects
@@
 			)
 		)
-		(property "LCSC" "C22374861"
+		(property "LCSC" "C22374841"
 			(at 191.77 87.63 0)
 			(effects
@@
 			)
 		)
+		(property "LCSC" "C3284550"
+			(at 267.97 87.63 0)
+			(effects
+				(font
+					(size 1.27 1.27)
+				)
+				(justify bottom)
+				(hide yes)
+			)
+		)
 		(property "Datasheet" ""
 			(at 267.97 87.63 0)
@@
 			)
 		)
-		(property "LCSC" "C381880"
+		(property "LCSC" "C52109780"
 			(at 138.43 106.68 0)
 			(effects
@@
 			)
 		)
-		(property "LCSC" "C778764"
+		(property "LCSC" "C52109745"
 			(at 166.37 82.55 90)
 			(effects
@@
 			)
 		)
-		(property "LCSC" "C32949"
+		(property "LCSC" "C387913"
 			(at 102.87 130.81 0)
 			(effects
@@
 			)
 		)
-		(property "LCSC" "C161321"
+		(property "LCSC" "C301911"
 			(at 251.46 95.25 0)
 			(effects
@@
 			)
 		)
-		(property "LCSC" "C1623"
+		(property "LCSC" "C7393835"
 			(at 39.37 110.49 0)
 			(effects
@@
 			)
 		)
-		(property "LCSC" "C86065"
+		(property "LCSC" "C52109761"
 			(at 186.69 82.55 90)
 			(effects
@@
 			)
 		)
-		(property "Value" "C_Small"
+		(property "Value" "NC"
 			(at 158.75 114.2935 0)
 			(effects
@@
 			)
 		)
-		(property "Value" "C_Small"
+		(property "Value" "NC"
 			(at 162.56 90.1635 0)
 			(effects

Commit message: Rev. C: schemafixes uit datasheetcontrole (VDD-buffer nRF9151, DC-blok LoRa, DNP C70/C71/BT2, deler 1M, laadtimers aan)
Parts:
- C70, C71: now not fitted; now left out of the parts list
- C96: renamed from R6; value 0R -> 56pF; footprint Resistor_SMD:R_0201_0603Metric -> Capacitor_SMD:C_0201_0603Metric; symbol Device:R_Small -> Device:C_Small; LCSC C473473 -> C2183491
Changed lines of the file:
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@@
 	)
 	(symbol
-		(lib_id "Device:R_Small")
+		(lib_id "Device:C_Small")
 		(at 232.41 90.17 90)
 		(unit 1)
@@
 		(dnp no)
 		(fields_autoplaced yes)
-		(property "Reference" "R6"
+		(property "Reference" "C96"
 			(at 232.41 85.09 90)
 			(effects
@@
 			)
 		)
-		(property "Value" "0R"
+		(property "Value" "56pF"
 			(at 232.41 87.63 90)
 			(effects
@@
 			)
 		)
-		(property "Footprint" "Resistor_SMD:R_0201_0603Metric"
+		(property "Footprint" "Capacitor_SMD:C_0201_0603Metric"
 			(at 232.41 90.17 0)
 			(effects
@@
 			)
 		)
-		(property "Datasheet" "https://jlcpcb.com/partdetail/25819-0402WGF1000TCE/C25076"
+		(property "Datasheet" ""
 			(at 232.41 90.17 0)
 			(effects
@@
 			)
 		)
-		(property "Description" "Resistor, small symbol"
+		(property "Description" "Unpolarized capacitor, small symbol"
 			(at 232.41 90.17 0)
 			(effects
@@
 			)
 		)
-		(property "LCSC" "C473473"
+		(property "LCSC" "C2183491"
 			(at 232.41 90.17 90)
 			(effects
@@
 			(project "Mesh3310"
 				(path "/8d65c5ef-7a02-4454-aee5-ab9c49e4aeab/d4d7259f-52be-4eaa-97bd-35f544c05202"
-					(reference "R6")
+					(reference "C96")
 					(unit 1)
 				)
@@
 		(unit 1)
 		(exclude_from_sim no)
-		(in_bom yes)
+		(in_bom no)
 		(on_board yes)
-		(dnp no)
+		(dnp yes)
 		(fields_autoplaced yes)
 		(property "Reference" "C70"
@@
 		(unit 1)
 		(exclude_from_sim no)
-		(in_bom yes)
+		(in_bom no)
 		(on_board yes)
-		(dnp no)
+		(dnp yes)
 		(fields_autoplaced yes)
 		(property "Reference" "C71"

Commit message: Rev. F + G: controleronde, TPS3420 aan/uit-knop, FLASH_CS pull-up, RF4 DNP, U.FL-variant LoRa
Parts:
- C81: value 3pF -> 3.3pF; LCSC C501815 -> C124777
- L16: footprint Inductor_SMD:L_0201_0603Metric -> Inductor_SMD:L_0402_1005Metric; LCSC C46607399 -> C192855
- RF4: now not fitted; now left out of the parts list
Changed lines of the file:
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@@
 		(title "Mainboard replacement for Nokia 3310")
 		(date "29-12-2025")
-		(rev "Rev A")
+		(rev "Rev G")
 		(company "Mesh3310")
 		(comment 1 "JDJ electronics")
@@
 			)
 		)
-		(property "Value" "3pF"
+		(property "Value" "3.3pF"
 			(at 166.3763 68.58 90)
 			(effects
@@
 			)
 		)
-		(property "LCSC" "C501815"
+		(property "LCSC" "C124777"
 			(at 166.37 72.39 90)
 			(effects
@@
 			)
 		)
-		(property "Footprint" "Inductor_SMD:L_0201_0603Metric"
+		(property "Footprint" "Inductor_SMD:L_0402_1005Metric"
 			(at 151.13 73.66 0)
 			(effects
@@
 			)
 		)
-		(property "LCSC" "C46607399"
+		(property "LCSC" "C192855"
 			(at 151.13 73.66 0)
 			(effects
@@
 		(unit 1)
 		(exclude_from_sim no)
-		(in_bom yes)
+		(in_bom no)
 		(on_board yes)
-		(dnp no)
+		(dnp yes)
 		(fields_autoplaced yes)
 		(property "Reference" "RF4"

Commit message: Onderdelen die JLC niet had vervangen, JLC-uploadbestanden toegevoegd
Parts:
- C75, C84: LCSC C22374841 -> C161416
- C81: LCSC C124777 -> C161425
Changed lines of the file:
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@@
 			)
 		)
-		(property "LCSC" "C124777"
+		(property "LCSC" "C161425"
 			(at 166.37 72.39 90)
 			(effects
@@
 			)
 		)
-		(property "LCSC" "C22374841"
+		(property "LCSC" "C161416"
 			(at 138.43 113.03 0)
 			(effects
@@
 			)
 		)
-		(property "LCSC" "C22374841"
+		(property "LCSC" "C161416"
 			(at 191.77 87.63 0)
 			(effects
